File: design/hv-bank.kicad_sch (KiCad schematic)
At the start: 0 parts

Commit message: started primary power distribution design
Other:
- company: (none) -> UNH Resilient Architecture Lab
- title: (none) -> BitCrusher: Affordable, Open Source EMFI Platform
Changed lines of the file:
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@@
 	(generator_version "9.0")
 	(paper "A4")
+	(title_block
+		(title "BitCrusher: Affordable, Open Source EMFI Platform")
+		(rev "0.1")
+		(company "UNH Resilient Architecture Lab")
+		(comment 1 "Author: George Crane")
+	)
 )
