File: design/power.kicad_sch (KiCad schematic)
At the start: 37 parts, among them J8 Barrel_Jack, U4 TPS7A2050PDQN, U5 TPS7A2033PDQN, U6 LMR33630ADDA, U7 LMR33630ADDA

Commit message: More footprint assignment and component selection
Parts:
- RFBB1, RFBB2, RFBT1, RFBT2, RPG1, RPG2: footprint Resistor_SMD:R_0402_1005Metric -> Resistor_SMD:R_2512_6332Metric
Changed lines of the file:
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@@
 			)
 		)
-		(property "Footprint" "Resistor_SMD:R_0402_1005Metric"
+		(property "Footprint" "Resistor_SMD:R_2512_6332Metric"
 			(at 45.72 131.318 90)
 			(effects
@@
 			)
 		)
-		(property "Footprint" "Resistor_SMD:R_0402_1005Metric"
+		(property "Footprint" "Resistor_SMD:R_2512_6332Metric"
 			(at 83.312 72.39 90)
 			(effects
@@
 			)
 		)
-		(property "Footprint" "Resistor_SMD:R_0402_1005Metric"
+		(property "Footprint" "Resistor_SMD:R_2512_6332Metric"
 			(at 45.72 77.978 90)
 			(effects
@@
 			)
 		)
-		(property "Footprint" "Resistor_SMD:R_0402_1005Metric"
+		(property "Footprint" "Resistor_SMD:R_2512_6332Metric"
 			(at 86.868 118.11 90)
 			(effects
@@
 			)
 		)
-		(property "Footprint" "Resistor_SMD:R_0402_1005Metric"
+		(property "Footprint" "Resistor_SMD:R_2512_6332Metric"
 			(at 86.868 64.77 90)
 			(effects
@@
 			)
 		)
-		(property "Footprint" "Resistor_SMD:R_0402_1005Metric"
+		(property "Footprint" "Resistor_SMD:R_2512_6332Metric"
 			(at 83.312 125.73 90)
 			(effects

Commit message: Done with component selection / footprint assignment
Parts:
- J8: value Barrel_Jack -> PJ-002BH; footprint (none) -> project-footprints:PJ-002B_CUI
Changed lines of the file:
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@@
 			)
 		)
-		(property "Value" "Barrel_Jack"
+		(property "Value" "PJ-002BH"
 			(at 21.59 17.78 0)
 			(effects
@@
 			)
 		)
-		(property "Footprint" ""
+		(property "Footprint" "project-footprints:PJ-002B_CUI"
 			(at 22.86 25.146 0)
 			(effects
@@
 			)
 		)
-		(property "Description" "DC Barrel Jack"
+		(property "Description" "5.5x2.5mm"
 			(at 21.59 24.13 0)
 			(effects

Commit message: Starting PCB layout
Parts:
- renumbered J8 to J10
Changed lines of the file:
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@@
 		(dnp no)
 		(fields_autoplaced yes)
-		(property "Reference" "#PWR019"
+		(property "Reference" "#PWR021"
 			(at 162.56 50.8 0)
 			(effects
@@
 			(project "BitCrusher"
 				(path "/e1be550d-9ce6-42b1-a89a-c00b9d7586dd/e3389efa-d643-4121-9f24-b7f22e7fe0ec"
-					(reference "#PWR019")
+					(reference "#PWR021")
 					(unit 1)
 				)
@@
 		(dnp no)
 		(fields_autoplaced yes)
-		(property "Reference" "J8"
+		(property "Reference" "J10"
 			(at 21.59 15.24 0)
 			(effects
@@
 			(project "BitCrusher"
 				(path "/e1be550d-9ce6-42b1-a89a-c00b9d7586dd/e3389efa-d643-4121-9f24-b7f22e7fe0ec"
-					(reference "J8")
+					(reference "J10")
 					(unit 1)
 				)
@@
 		(dnp no)
 		(fields_autoplaced yes)
-		(property "Reference" "#PWR024"
+		(property "Reference" "#PWR026"
 			(at 140.97 60.96 0)
 			(effects
@@
 			(project "BitCrusher"
 				(path "/e1be550d-9ce6-42b1-a89a-c00b9d7586dd/e3389efa-d643-4121-9f24-b7f22e7fe0ec"
-					(reference "#PWR024")
+					(reference "#PWR026")
 					(unit 1)
 				)
@@
 		(dnp no)
 		(fields_autoplaced yes)
-		(property "Reference" "#PWR022"
+		(property "Reference" "#PWR024"
 			(at 229.87 50.8 0)
 			(effects
@@
 			(project "BitCrusher"
 				(path "/e1be550d-9ce6-42b1-a89a-c00b9d7586dd/e3389efa-d643-4121-9f24-b7f22e7fe0ec"
-					(reference "#PWR022")
+					(reference "#PWR024")
 					(unit 1)
 				)
@@
 		(dnp no)
 		(fields_autoplaced yes)
-		(property "Reference" "#PWR021"
+		(property "Reference" "#PWR023"
 			(at 204.47 50.8 0)
 			(effects
@@
 			(project "BitCrusher"
 				(path "/e1be550d-9ce6-42b1-a89a-c00b9d7586dd/e3389efa-d643-4121-9f24-b7f22e7fe0ec"
-					(reference "#PWR021")
+					(reference "#PWR023")
 					(unit 1)
 				)
@@
 		(dnp no)
 		(fields_autoplaced yes)
-		(property "Reference" "#PWR026"
+		(property "Reference" "#PWR028"
 			(at 140.97 114.3 0)
 			(effects
@@
 			(project "BitCrusher"
 				(path "/e1be550d-9ce6-42b1-a89a-c00b9d7586dd/e3389efa-d643-4121-9f24-b7f22e7fe0ec"
-					(reference "#PWR026")
+					(reference "#PWR028")
 					(unit 1)
 				)
@@
 		(dnp no)
 		(fields_autoplaced yes)
-		(property "Reference" "#PWR020"
+		(property "Reference" "#PWR022"
 			(at 190.5 50.8 0)
 			(effects
@@
 			(project "BitCrusher"
 				(path "/e1be550d-9ce6-42b1-a89a-c00b9d7586dd/e3389efa-d643-4121-9f24-b7f22e7fe0ec"
-					(reference "#PWR020")
+					(reference "#PWR022")
 					(unit 1)
 				)
@@
 		(dnp no)
 		(fields_autoplaced yes)
-		(property "Reference" "#PWR023"
+		(property "Reference" "#PWR025"
 			(at 236.22 50.8 0)
 			(effects
@@
 			(project "BitCrusher"
 				(path "/e1be550d-9ce6-42b1-a89a-c00b9d7586dd/e3389efa-d643-4121-9f24-b7f22e7fe0ec"
-					(reference "#PWR023")
+					(reference "#PWR025")
 					(unit 1)
 				)
@@
 		(dnp no)
 		(fields_autoplaced yes)
-		(property "Reference" "#PWR025"
+		(property "Reference" "#PWR027"
 			(at 35.56 104.14 0)
 			(effects
@@
 			(project "BitCrusher"
 				(path "/e1be550d-9ce6-42b1-a89a-c00b9d7586dd/e3389efa-d643-4121-9f24-b7f22e7fe0ec"
-					(reference "#PWR025")
+					(reference "#PWR027")
 					(unit 1)
 				)

Commit message: Primary power layout
Parts:
- RFBB1, RFBB2, RFBT1, RFBT2, RPG1, RPG2: footprint Resistor_SMD:R_2512_6332Metric -> Resistor_SMD:R_0603_1608Metric
Changed lines of the file:
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@@
 			)
 		)
-		(property "Footprint" "Resistor_SMD:R_2512_6332Metric"
+		(property "Footprint" "Resistor_SMD:R_0603_1608Metric"
 			(at 45.72 131.318 90)
 			(effects
@@
 			)
 		)
-		(property "Footprint" "Resistor_SMD:R_2512_6332Metric"
+		(property "Footprint" "Resistor_SMD:R_0603_1608Metric"
 			(at 83.312 72.39 90)
 			(effects
@@
 			)
 		)
-		(property "Footprint" "Resistor_SMD:R_2512_6332Metric"
+		(property "Footprint" "Resistor_SMD:R_0603_1608Metric"
 			(at 45.72 77.978 90)
 			(effects
@@
 			)
 		)
-		(property "Footprint" "Resistor_SMD:R_2512_6332Metric"
+		(property "Footprint" "Resistor_SMD:R_0603_1608Metric"
 			(at 86.868 118.11 90)
 			(effects
@@
 			)
 		)
-		(property "Footprint" "Resistor_SMD:R_2512_6332Metric"
+		(property "Footprint" "Resistor_SMD:R_0603_1608Metric"
 			(at 86.868 64.77 90)
 			(effects
@@
 			)
 		)
-		(property "Footprint" "Resistor_SMD:R_2512_6332Metric"
+		(property "Footprint" "Resistor_SMD:R_0603_1608Metric"
 			(at 83.312 125.73 90)
 			(effects

Commit message: Fixing layout and parts selection issues for prototype run
Parts:
- L1: value 15.4u -> 15u
Changed lines of the file:
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@@
 			)
 		)
-		(property "Value" "15.4u"
+		(property "Value" "15u"
 			(at 80.01 55.88 90)
 			(effects
@@
 			)
 		)
-		(property "Description" "SL0630-100M 10uH 5.5A 5A ±20% SMD,7.1x6.6mm Inductors (SMD) ROHS"
+		(property "Description" "SL0630-150M"
 			(at 80.01 58.42 0)
 			(effects

Commit message: _
Other:
- note removed: "Should support a peak current of the flyback converter I_peak (2A)+10% (2.2A)"

Commit message: Added missing 3d models
Parts:
- U6, U7: footprint Package_SO:Texas_HSOP-8-1EP_3.9x4.9mm_P1.27mm_ThermalVias -> project-footprints:Texas_HSOP-8-1EP_3.9x4.9mm_P1.27mm_ThermalVias
Changed lines of the file:
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@@
 			)
 		)
-		(property "Footprint" "Package_SO:Texas_HSOP-8-1EP_3.9x4.9mm_P1.27mm_ThermalVias"
+		(property "Footprint" "project-footprints:Texas_HSOP-8-1EP_3.9x4.9mm_P1.27mm_ThermalVias"
 			(at 46.99 134.62 0)
 			(effects
@@
 			)
 		)
-		(property "Footprint" "Package_SO:Texas_HSOP-8-1EP_3.9x4.9mm_P1.27mm_ThermalVias"
+		(property "Footprint" "project-footprints:Texas_HSOP-8-1EP_3.9x4.9mm_P1.27mm_ThermalVias"
 			(at 46.99 81.28 0)
 			(effects
