File: design/control.kicad_sch (KiCad schematic)
At the start: 29 parts, among them J1 USB_C_Receptacle_USB2.0_14P, J2 SMB, J3 Conn-OScope, J4 Conn-OScope, J5 SMA, J7 Conn_01x02_Pin, J8 Conn_01x02_Pin, U2 STM32F303RETx, U6 USBLC6-2SC6, U8 FT230XQ

Commit message: _
Parts:
- R22, R23: footprint (none) -> Resistor_SMD:R_0402_1005Metric
Other:
- note added: "DAC1_OUT1 (3V)"
- note removed: "DAC1_OUT1"
Changed lines of the file:
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@@
 		)
 	)
-	(text "DAC1_OUT1"
+	(text "DAC1_OUT1 (3V)"
 		(exclude_from_sim no)
 		(at 216.408 59.944 0)
@@
 			)
 		)
-		(property "Footprint" ""
+		(property "Footprint" "Resistor_SMD:R_0402_1005Metric"
 			(at 113.03 132.842 90)
 			(effects
@@
 			)
 		)
-		(property "Footprint" ""
+		(property "Footprint" "Resistor_SMD:R_0402_1005Metric"
 			(at 102.87 132.842 90)
 			(effects

Commit message: Footprint assignment / part selection
Parts:
- renumbered C28 to C10, C29 to C11, C27 to C12, C4 to C3, C5 to C4, C6 to C5, C7 to C6, C8 to C7, C3 to C8, C26 to C9, D8 to D1, D9 to D2, J2 to J1, J5 to J2, J1 to J5, J7 to J6, J8 to J7, R5 to R1, R1 to R2, R2 to R3, R22 to R4, R23 to R5, U2 to U1, U6 to U2, U8 to U3

Commit message: More footprint assignment and component selection
Parts:
- J1: value SMB -> BNC; footprint (none) -> project-footprints:KHBNC503511
- J2: value SMA -> BWSMA-KWE-Z001; footprint (none) -> Connector_Coaxial:SMA_BAT_Wireless_BWSMA-KWE-Z001
- J3, J4: value Conn-OScope -> BWSMA-KE-Z001; footprint (none) -> project-footprints:SMA_BAT_Wireless_BWSMA-KE-Z001
Changed lines of the file:
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@@
 	(rectangle
 		(start 19.05 20.32)
-		(end 90.17 63.5)
+		(end 94.615 63.5)
 		(stroke
 			(width 0)
@@
 			)
 		)
-		(property "Value" "SMB"
+		(property "Value" "BNC"
 			(at 44.45 26.9631 0)
 			(effects
@@
 			)
 		)
-		(property "Footprint" ""
+		(property "Footprint" "project-footprints:KHBNC503511"
 			(at 40.64 25.4 0)
 			(effects
@@
 			)
 		)
-		(property "Value" "Conn-OScope"
+		(property "Value" "BWSMA-KE-Z001"
 			(at 74.93 52.3631 0)
 			(effects
@@
 			)
 		)
-		(property "Footprint" ""
+		(property "Footprint" "project-footprints:SMA_BAT_Wireless_BWSMA-KE-Z001"
 			(at 71.12 50.8 0)
 			(effects
@@
 			)
 		)
-		(property "Value" "Conn-OScope"
+		(property "Value" "BWSMA-KE-Z001"
 			(at 74.93 38.3931 0)
 			(effects
@@
 			)
 		)
-		(property "Footprint" ""
+		(property "Footprint" "project-footprints:SMA_BAT_Wireless_BWSMA-KE-Z001"
 			(at 71.12 36.83 0)
 			(effects
@@
 			)
 		)
-		(property "Value" "SMA"
+		(property "Value" "BWSMA-KWE-Z001"
 			(at 74.93 26.9631 0)
 			(effects
@@
 			)
 		)
-		(property "Footprint" ""
+		(property "Footprint" "Connector_Coaxial:SMA_BAT_Wireless_BWSMA-KWE-Z001"
 			(at 71.12 25.4 0)
 			(effects

Commit message: More footprint assignment (almost done)
Connections:
- net GNDHV: no longer D1.1 (A1), J3.2 (Ext)
- net ADC1_IN2 renamed HVVS-
- net ADC1_IN4 renamed PulseVS-
- net PulseVS-: now also D1.1 (A1), J3.2 (Ext)
- net HVVS renamed HVVS+
- net PulseVS renamed PulseVS+
Changed lines of the file:
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@@
 		)
 	)
-	(global_label "HVVS"
+	(global_label "HVVS+"
 		(shape input)
 		(at 224.79 49.53 0)
@@
 		)
 		(property "Intersheetrefs" "${INTERSHEET_REFS}"
-			(at 232.4924 49.53 0)
+			(at 234.0648 49.53 0)
 			(effects
 				(font
@@
 		)
 	)
-	(global_label "PulseVS"
+	(global_label "PulseVS+"
 		(shape input)
 		(at 60.96 36.83 180)
@@
 		)
 		(property "Intersheetrefs" "${INTERSHEET_REFS}"
-			(at 50.4758 36.83 0)
+			(at 48.9034 36.83 0)
 			(effects
 				(font
@@
 		)
 	)
-	(global_label "ADC1_IN4"
+	(global_label "PulseVS-"
 		(shape input)
 		(at 224.79 57.15 0)
@@
 		)
 		(property "Intersheetrefs" "${INTERSHEET_REFS}"
-			(at 236.7257 57.15 0)
+			(at 236.8466 57.15 0)
 			(effects
 				(font
@@
 		)
 	)
-	(global_label "ADC1_IN2"
+	(global_label "HVVS-"
 		(shape input)
 		(at 224.79 52.07 0)
@@
 		)
 		(property "Intersheetrefs" "${INTERSHEET_REFS}"
-			(at 236.7257 52.07 0)
+			(at 234.0648 52.07 0)
 			(effects
 				(font
@@
 		)
 	)
-	(global_label "PulseVS"
+	(global_label "PulseVS+"
 		(shape input)
 		(at 224.79 54.61 0)
@@
 		)
 		(property "Intersheetrefs" "${INTERSHEET_REFS}"
-			(at 235.2742 54.61 0)
+			(at 236.8466 54.61 0)
 			(effects
 				(font
@@
 		)
 	)
+	(global_label "PulseVS-"
+		(shape input)
+		(at 60.96 44.45 180)
+		(fields_autoplaced yes)
+		(effects
+			(font
+				(size 1.27 1.27)
+			)
+			(justify right)
+		)
+		(property "Intersheetrefs" "${INTERSHEET_REFS}"
+			(at 48.9034 44.45 0)
+			(effects
+				(font
+					(size 1.27 1.27)
+				)
+				(justify right)
+				(hide yes)
+			)
+		)
+	)
 	(global_label "USART1_TX"
 		(shape input)
@@
 					(unit 1)
 				)
-			)
-		)
-	)
-	(symbol
-		(lib_id "power:GNDPWR")
-		(at 60.96 44.45 0)
-		(unit 1)
-		(exclude_from_sim no)
-		(in_bom yes)
-		(on_board yes)
-		(dnp no)
-		(fields_autoplaced yes)
-		(property "Reference" "#PWR06"
-			(at 60.96 49.53 0)
-			(effects
-				(font
-					(size 1.27 1.27)
-				)
-				(hide yes)
-			)
-		)
-		(property "Value" "GNDHV"
-			(at 60.833 48.26 0)
-			(effects
-				(font
-					(size 1.27 1.27)
-				)
-			)
-		)
-		(property "Footprint" ""
-			(at 60.96 45.72 0)
-			(effects
-				(font
-					(size 1.27 1.27)
-				)
-				(hide yes)
-			)
-		)
-		(property "Datasheet" ""
-			(at 60.96 45.72 0)
-			(effects
-				(font
-					(size 1.27 1.27)
-				)
-				(hide yes)
-			)
-		)
-		(property "Description" "Power symbol creates a global label with name \"GNDPWR\" , global ground"
-			(at 60.96 44.45 0)
-			(effects
-				(font
-					(size 1.27 1.27)
-				)
-				(hide yes)
-			)
-		)
-		(pin "1"
-		)
-		(instances
-			(project "BitCrusher"
-				(path "/e1be550d-9ce6-42b1-a89a-c00b9d7586dd/29f45a98-1f25-4a6e-8231-3aa3a650ea17"
-					(reference "#PWR06")
-					(unit 1)
-				)

Commit message: Done with component selection / footprint assignment
Parts:
- removed J6, J7: Conn_01x02_Pin, Connector_PinHeader_2.54mm:PinHeader_1x02_P2.54mm_Vertical, symbol Connector:Conn_01x02_Pin
- added J10, J6: Conn_01x03_Pin, Connector_PinHeader_2.54mm:PinHeader_1x03_P2.54mm_Vertical, symbol Connector:Conn_01x03_Pin
- added J9: Conn_01x04_Pin, Connector_PinHeader_2.54mm:PinHeader_1x04_P2.54mm_Vertical, symbol Connector:Conn_01x04_Pin
- J5: value USB_C_Receptacle_USB2.0_14P -> SHOU HAN TYPE-C 14P CC-2.6; footprint (none) -> project-footprints:TYPE-C-TH_TYPE-C-14P-CC-2.6
Connections:
- net +3V3: now also J10.1 (Pin_1), J6.1 (Pin_1)
- net BOOTSEL: now also J10.2 (Pin_2)
- net GND: now also J10.3 (Pin_3), J6.3 (Pin_3)
- net PulseVS+: no longer U1.16 (PA2)
- net PulseVS-: no longer U1.17 (PA3)
- net RST: now also J6.2 (Pin_2)
- net USART1_RX: now also J9.4 (Pin_4); no longer U3.15 (TXD)
- net USART1_TX: now also J9.1 (Pin_1); no longer U3.2 (RXD)
- net GNDHV renamed PulseCS-
- net PulseCS renamed PulseCS+
- new net RX_IN: J9.3 (Pin_3), U3.15 (TXD)
- new net TX_IN: J9.2 (Pin_2), U3.2 (RXD)
- no-connect marks 4 -> 45
Other:
- note added: "Debugging Interfaces / Jumpers"
- note removed: "Open drain"
- note removed: "Push pull"

Commit message: Cleanup
Parts:
- added J7: Conn_01x04_Pin, Connector_PinHeader_2.54mm:PinHeader_1x04_P2.54mm_Vertical, symbol Connector:Conn_01x04_Pin
Connections:
- net PulseEN: now also U1.44 (PA11); no longer U1.61 (PB8)
- net Debug1: now reaches U1.55 (PB3)
- net Debug1: now also J7.1 (Pin_1)
- net Debug2: now reaches U1.56 (PB4)
- net Debug2: now also J7.2 (Pin_2)
- net Debug3: now reaches U1.57 (PB5)
- net Debug3: now also J7.3 (Pin_3)
- net Debug4: now reaches U1.58 (PB6)
- net Debug4: now also J7.4 (Pin_4)
- no-connect marks 45 -> 40
Other:
- note added: "DAC1_OUT1"
- note removed: "ADC1_IN3"
- note removed: "ADC1_IN4"
- note removed: "Breakout some extra GPIOs"
- note removed: "DAC1_OUT1 (3V)"

Commit message: Starting PCB layout
Parts:
- renumbered J9 to J6, J6 to J8, J10 to J9
Changed lines of the file:
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@@
 		(dnp no)
 		(fields_autoplaced yes)
-		(property "Reference" "#PWR09"
+		(property "Reference" "#PWR07"
 			(at 55.88 77.47 0)
 			(effects
@@
 			(project "BitCrusher"
 				(path "/e1be550d-9ce6-42b1-a89a-c00b9d7586dd/29f45a98-1f25-4a6e-8231-3aa3a650ea17"
-					(reference "#PWR09")
+					(reference "#PWR07")
 					(unit 1)
 				)
@@
 		(dnp no)
 		(fields_autoplaced yes)
-		(property "Reference" "#PWR018"
+		(property "Reference" "#PWR016"
 			(at 196.85 147.32 0)
 			(effects
@@
 			(project ""
 				(path "/e1be550d-9ce6-42b1-a89a-c00b9d7586dd/29f45a98-1f25-4a6e-8231-3aa3a650ea17"
-					(reference "#PWR018")
+					(reference "#PWR016")
 					(unit 1)
 				)
@@
 		(dnp no)
 		(fields_autoplaced yes)
-		(property "Reference" "#PWR044"
+		(property "Reference" "#PWR018"
 			(at 59.69 175.26 0)
 			(effects
@@
 			(project "BitCrusher"
 				(path "/e1be550d-9ce6-42b1-a89a-c00b9d7586dd/29f45a98-1f25-4a6e-8231-3aa3a650ea17"
-					(reference "#PWR044")
+					(reference "#PWR018")
 					(unit 1)
 				)
@@
 		(dnp no)
 		(fields_autoplaced yes)
-		(property "Reference" "#PWR046"
+		(property "Reference" "#PWR020"
 			(at 59.69 193.04 0)
 			(effects
@@
 			(project "BitCrusher"
 				(path "/e1be550d-9ce6-42b1-a89a-c00b9d7586dd/29f45a98-1f25-4a6e-8231-3aa3a650ea17"
-					(reference "#PWR046")
+					(reference "#PWR020")
 					(unit 1)
 				)
@@
 		(dnp no)
 		(fields_autoplaced yes)
-		(property "Reference" "J10"
+		(property "Reference" "J9"
 			(at 67.31 181.6099 0)
 			(effects
@@
 			(project "BitCrusher"
 				(path "/e1be550d-9ce6-42b1-a89a-c00b9d7586dd/29f45a98-1f25-4a6e-8231-3aa3a650ea17"
-					(reference "J10")
+					(reference "J9")
 					(unit 1)
 				)
@@
 		(dnp no)
 		(fields_autoplaced yes)
-		(property "Reference" "#PWR013"
+		(property "Reference" "#PWR011"
 			(at 68.58 120.65 0)
 			(effects
@@
 			(project "BitCrusher"
 				(path "/e1be550d-9ce6-42b1-a89a-c00b9d7586dd/29f45a98-1f25-4a6e-8231-3aa3a650ea17"
-					(reference "#PWR013")
+					(reference "#PWR011")
 					(unit 1)
 				)
@@
 		(dnp no)
 		(fields_autoplaced yes)
-		(property "Reference" "J9"
+		(property "Reference" "J6"
 			(at 36.83 163.8299 0)
 			(effects
@@
 			(project ""
 				(path "/e1be550d-9ce6-42b1-a89a-c00b9d7586dd/29f45a98-1f25-4a6e-8231-3aa3a650ea17"
-					(reference "J9")
+					(reference "J6")
 					(unit 1)
 				)
@@
 		(dnp no)
 		(fields_autoplaced yes)
-		(property "Reference" "J6"
+		(property "Reference" "J8"
 			(at 67.31 163.8299 0)
 			(effects
@@
 			(project ""
 				(path "/e1be550d-9ce6-42b1-a89a-c00b9d7586dd/29f45a98-1f25-4a6e-8231-3aa3a650ea17"
-					(reference "J6")
+					(reference "J8")
 					(unit 1)
 				)
@@
 		(dnp no)
 		(fields_autoplaced yes)
-		(property "Reference" "#PWR08"
+		(property "Reference" "#PWR06"
 			(at 146.05 66.04 0)
 			(effects
@@
 			(project "BitCrusher"
 				(path "/e1be550d-9ce6-42b1-a89a-c00b9d7586dd/29f45a98-1f25-4a6e-8231-3aa3a650ea17"
-					(reference "#PWR08")
+					(reference "#PWR06")
 					(unit 1)
 				)
@@
 		(dnp no)
 		(fields_autoplaced yes)
-		(property "Reference" "#PWR016"
+		(property "Reference" "#PWR014"
 			(at 31.75 135.89 0)
 			(effects
@@
 			(project "BitCrusher"
 				(path "/e1be550d-9ce6-42b1-a89a-c00b9d7586dd/29f45a98-1f25-4a6e-8231-3aa3a650ea17"
-					(reference "#PWR016")
+					(reference "#PWR014")
 					(unit 1)
 				)
@@
 		(dnp no)
 		(fields_autoplaced yes)
-		(property "Reference" "#PWR014"
+		(property "Reference" "#PWR012"
 			(at 93.98 133.35 0)
 			(effects
@@
 			(project "BitCrusher"
 				(path "/e1be550d-9ce6-42b1-a89a-c00b9d7586dd/29f45a98-1f25-4a6e-8231-3aa3a650ea17"
-					(reference "#PWR014")
+					(reference "#PWR012")
 					(unit 1)
 				)
@@
 		(dnp no)
 		(fields_autoplaced yes)
-		(property "Reference" "#PWR017"
+		(property "Reference" "#PWR015"
 			(at 118.11 142.24 0)
 			(effects
@@
 			(project "BitCrusher"
 				(path "/e1be550d-9ce6-42b1-a89a-c00b9d7586dd/29f45a98-1f25-4a6e-8231-3aa3a650ea17"
-					(reference "#PWR017")
+					(reference "#PWR015")
 					(unit 1)
 				)
@@
 		(dnp no)
 		(fields_autoplaced yes)
-		(property "Reference" "#PWR015"
+		(property "Reference" "#PWR013"
 			(at 24.13 135.89 0)
 			(effects
@@
 			(project "BitCrusher"
 				(path "/e1be550d-9ce6-42b1-a89a-c00b9d7586dd/29f45a98-1f25-4a6e-8231-3aa3a650ea17"
-					(reference "#PWR015")
+					(reference "#PWR013")
 					(unit 1)
 				)
@@
 		(dnp no)
 		(fields_autoplaced yes)
-		(property "Reference" "#PWR07"
+		(property "Reference" "#PWR017"
 			(at 59.69 165.1 0)
 			(effects
@@
 			(project "BitCrusher"
 				(path "/e1be550d-9ce6-42b1-a89a-c00b9d7586dd/29f45a98-1f25-4a6e-8231-3aa3a650ea17"
-					(reference "#PWR07")
+					(reference "#PWR017")
 					(unit 1)
 				)
@@
 		(dnp no)
 		(fields_autoplaced yes)
-		(property "Reference" "#PWR010"
+		(property "Reference" "#PWR08"
 			(at 64.77 93.98 0)
 			(effects
@@
 			(project "BitCrusher"
 				(path "/e1be550d-9ce6-42b1-a89a-c00b9d7586dd/29f45a98-1f25-4a6e-8231-3aa3a650ea17"
-					(reference "#PWR010")
+					(reference "#PWR08")
 					(unit 1)
 				)
@@
 		(on_board yes)
 		(dnp no)
-		(property "Reference" "#PWR045"
+		(property "Reference" "#PWR019"
 			(at 59.69 182.88 0)
 			(effects
@@
 			(project "BitCrusher"
 				(path "/e1be550d-9ce6-42b1-a89a-c00b9d7586dd/29f45a98-1f25-4a6e-8231-3aa3a650ea17"
-					(reference "#PWR045")
+					(reference "#PWR019")
 					(unit 1)
 				)
@@
 		(dnp no)
 		(fields_autoplaced yes)
-		(property "Reference" "#PWR011"
+		(property "Reference" "#PWR09"
 			(at 101.6 99.06 0)
 			(effects
@@
 			(project "BitCrusher"
 				(path "/e1be550d-9ce6-42b1-a89a-c00b9d7586dd/29f45a98-1f25-4a6e-8231-3aa3a650ea17"
-					(reference "#PWR011")
+					(reference "#PWR09")
 					(unit 1)
 				)
@@
 		(dnp no)
 		(fields_autoplaced yes)
-		(property "Reference" "#PWR012"
+		(property "Reference" "#PWR010"
 			(at 63.5 106.68 0)
 			(effects
@@
 			(project "BitCrusher"
 				(path "/e1be550d-9ce6-42b1-a89a-c00b9d7586dd/29f45a98-1f25-4a6e-8231-3aa3a650ea17"
-					(reference "#PWR012")
+					(reference "#PWR010")
 					(unit 1)
 				)

Commit message: More layout work
Parts:
- added J11: Conn_01x04_Pin, Connector_PinHeader_2.54mm:PinHeader_1x04_P2.54mm_Vertical, symbol Connector:Conn_01x04_Pin
Connections:
- no-connect marks 40 -> 41
Changed lines of the file:
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@@
 	)
 	(no_connect
+		(at 214.63 113.03)
+	)
+	(no_connect
 		(at 214.63 72.39)
 	)
@@
 					(unit 1)
 				)
+			)
+		)
+	)
+	(symbol
+		(lib_id "Connector:Conn_01x04_Pin")
+		(at 101.6 179.07 0)
+		(mirror y)
+		(unit 1)
+		(exclude_from_sim no)
+		(in_bom yes)
+		(on_board yes)
+		(dnp no)
+		(fields_autoplaced yes)
+		(property "Reference" "J11"
+			(at 102.87 179.0699 0)
+			(effects
+				(font
+					(size 1.27 1.27)
+				)
+				(justify right)
+			)
+		)
+		(property "Value" "Conn_01x04_Pin"
+			(at 102.87 181.6099 0)
+			(effects
+				(font
+					(size 1.27 1.27)
+				)
+				(justify right)
+			)
+		)
+		(property "Footprint" "Connector_PinHeader_2.54mm:PinHeader_1x04_P2.54mm_Vertical"
+			(at 101.6 179.07 0)
+			(effects
+				(font
+					(size 1.27 1.27)
+				)
+				(hide yes)
+			)
+		)
+		(property "Datasheet" "~"
+			(at 101.6 179.07 0)
+			(effects
+				(font
+					(size 1.27 1.27)
+				)
+				(hide yes)
+			)
+		)
+		(property "Description" "Generic connector, single row, 01x04, script generated"
+			(at 101.6 179.07 0)
+			(effects
+				(font
+					(size 1.27 1.27)
+				)
+				(hide yes)
+			)
+		)
+		(pin "2"
+		)
+		(pin "1"
+		)
+		(pin "3"
+		)
+		(pin "4"
+		)
+		(instances
+			(project "BitCrusher"
+				(path "/e1be550d-9ce6-42b1-a89a-c00b9d7586dd/29f45a98-1f25-4a6e-8231-3aa3a650ea17"
+					(reference "J11")
+					(unit 1)
+				)
