File: design/hv-switch.kicad_sch (KiCad schematic)
At the start: 30 parts, among them Q3 GAN080-650EBE, U9 MAX22702EASA+

Commit message: Done with component selection / footprint assignment
Parts:
- removed D6: D, symbol Device:D
- added D6: 1N5822, Diode_THT:D_DO-201AD_P12.70mm_Horizontal, symbol Device:D_Schottky
Connections:
- net +6V: now also D6.2 (A)
- net at C27.1, C28.1, C29.1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: now also D6.1 (K)
- net PulseCS renamed PulseCS+
Changed lines of the file:
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@@
 	(wire
 		(pts
-			(xy 207.01 151.13) (xy 209.55 151.13)
+			(xy 203.2 151.13) (xy 209.55 151.13)
 		)
 		(stroke
@@
 	(wire
 		(pts
+			(xy 203.2 154.94) (xy 205.74 154.94)
+		)
+		(stroke
+			(width 0)
+			(type default)
+		)
+	)
+	(wire
+		(pts
 			(xy 195.58 119.38) (xy 201.93 119.38)
 		)
@@
 	(wire
 		(pts
+			(xy 205.74 154.94) (xy 205.74 157.48)
+		)
+		(stroke
+			(width 0)
+			(type default)
+		)
+	)
+	(wire
+		(pts
 			(xy 135.89 81.28) (xy 135.89 78.74)
 		)
@@
 		)
 	)
+	(global_label "PulseCS-"
+		(shape output)
+		(at 203.2 154.94 180)
+		(fields_autoplaced yes)
+		(effects
+			(font
+				(size 1.27 1.27)
+			)
+			(justify right)
+		)
+		(property "Intersheetrefs" "${INTERSHEET_REFS}"
+			(at 190.962 154.94 0)
+			(effects
+				(font
+					(size 1.27 1.27)
+				)
+				(justify right)
+				(hide yes)
+			)
+		)
+	)
 	(global_label "PulseEN"
 		(shape input)
@@
 		)
 	)
-	(global_label "PulseCS"
+	(global_label "PulseCS+"
 		(shape output)
-		(at 207.01 151.13 180)
+		(at 203.2 151.13 180)
 		(fields_autoplaced yes)
 		(effects
@@
 		)
 		(property "Intersheetrefs" "${INTERSHEET_REFS}"
-			(at 196.3444 151.13 0)
+			(at 190.962 151.13 0)
 			(effects
 				(font
@@
 	)
 	(symbol
+		(lib_id "Device:D_Schottky")
+		(at 111.76 35.56 90)
+		(unit 1)
+		(exclude_from_sim no)
+		(in_bom yes)
+		(on_board yes)
+		(dnp no)
+		(fields_autoplaced yes)
+		(property "Reference" "D6"
+			(at 114.3 34.6074 90)
+			(effects
+				(font
+					(size 1.27 1.27)
+				)
+				(justify right)
+			)
+		)
+		(property "Value" "1N5822"
+			(at 114.3 37.1474 90)
+			(effects
+				(font
+					(size 1.27 1.27)
+				)
+				(justify right)
+			)
+		)
+		(property "Footprint" "Diode_THT:D_DO-201AD_P12.70mm_Horizontal"
+			(at 111.76 35.56 0)
+			(effects
+				(font
+					(size 1.27 1.27)
+				)
+				(hide yes)
+			)
+		)
+		(property "Datasheet" "~"
+			(at 111.76 35.56 0)
+			(effects
+				(font
+					(size 1.27 1.27)
+				)
+				(hide yes)
+			)
+		)
+		(property "Description" "Schottky diode"
+			(at 111.76 35.56 0)
+			(effects
+				(font
+					(size 1.27 1.27)
+				)
+				(hide yes)
+			)
+		)
+		(property "Sim.Device" "D"
+			(at 111.76 35.56 0)
+			(effects
+				(font
+					(size 1.27 1.27)
+				)
+				(hide yes)
+			)
+		)
+		(property "Sim.Pins" "1=K 2=A"
+			(at 111.76 35.56 0)
+			(effects
+				(font
+					(size 1.27 1.27)
+				)
+				(hide yes)
+			)
+		)
+		(pin "2"
+		)
+		(pin "1"
+		)
+		(instances
+			(project "BitCrusher"
+				(path "/e1be550d-9ce6-42b1-a89a-c00b9d7586dd/a0344160-5a1e-4ade-9868-d857907b9d6d"
+					(reference "D6")
+					(unit 1)
+				)
+			)
+		)
+	)
+	(symbol
 		(lib_id "power:VDD")
 		(at 111.76 29.21 0)
@@
 	)
 	(symbol
-		(lib_id "Device:D")
-		(at 111.76 35.56 90)
+		(lib_id "power:GNDPWR")
+		(at 205.74 157.48 0)
 		(unit 1)
 		(exclude_from_sim no)
@@
 		(dnp no)
 		(fields_autoplaced yes)
-		(property "Reference" "D6"
-			(at 114.3 34.2899 90)
-			(effects
-				(font
-					(size 1.27 1.27)
-				)
-				(justify right)
-			)
-		)
-		(property "Value" "D"
-			(at 114.3 36.8299 90)
-			(effects
-				(font
-					(size 1.27 1.27)
-				)
-				(justify right)
-			)
-		)
-		(property "Footprint" ""
-			(at 111.76 35.56 0)
+		(property "Reference" "#PWR06"
+			(at 205.74 162.56 0)
 			(effects
 				(font
@@
 			)
 		)
-		(property "Datasheet" "~"
-			(at 111.76 35.56 0)
+		(property "Value" "GNDHV"
+			(at 205.613 161.29 0)
 			(effects
 				(font
 					(size 1.27 1.27)
 				)
-				(hide yes)
 			)
 		)
-		(property "Description" "Diode"
-			(at 111.76 35.56 0)
+		(property "Footprint" ""
+			(at 205.74 158.75 0)
 			(effects
 				(font
@@
 			)
 		)
-		(property "Sim.Device" "D"
-			(at 111.76 35.56 0)
+		(property "Datasheet" ""
+			(at 205.74 158.75 0)
 			(effects
 				(font
@@
 			)
 		)
-		(property "Sim.Pins" "1=K 2=A"
-			(at 111.76 35.56 0)
+		(property "Description" "Power symbol creates a global label with name \"GNDPWR\" , global ground"
+			(at 205.74 157.48 0)
 			(effects
 				(font
@@
 			)
 		)
-		(pin "2"
-		)
 		(pin "1"
 		)
 		(instances
-			(project ""
+			(project "BitCrusher"
 				(path "/e1be550d-9ce6-42b1-a89a-c00b9d7586dd/a0344160-5a1e-4ade-9868-d857907b9d6d"
-					(reference "D6")
+					(reference "#PWR06")
 					(unit 1)
 				)

Commit message: _
Parts:
- R20, R23, R24: footprint Resistor_SMD:R_2512_6332Metric -> Resistor_SMD:R_0603_1608Metric
Changed lines of the file:
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@@
 			)
 		)
-		(property "Footprint" "Resistor_SMD:R_2512_6332Metric"
+		(property "Footprint" "Resistor_SMD:R_0603_1608Metric"
 			(at 257.81 104.902 90)
 			(effects
@@
 			)
 		)
-		(property "Footprint" "Resistor_SMD:R_2512_6332Metric"
+		(property "Footprint" "Resistor_SMD:R_0603_1608Metric"
 			(at 215.9 149.352 90)
 			(effects
@@
 			)
 		)
-		(property "Footprint" "Resistor_SMD:R_2512_6332Metric"
+		(property "Footprint" "Resistor_SMD:R_0603_1608Metric"
 			(at 226.06 149.352 90)
 			(effects

Commit message: Fixing layout and parts selection issues for prototype run
Parts:
- added RP_B1: WSHP2818R0200FEA, project-footprints:WSHP2818R0200FEA, symbol Device:R
- added RP_LIM1: PF2472-0R1F1, Package_TO_SOT_THT:TO-247-2_Horizontal_TabDown, symbol Device:R
- C30: footprint Capacitor_SMD:C_0402_1005Metric -> Capacitor_SMD:C_0603_1608Metric
Connections:
- net GNDHV: now also RP_B1.1
- net Probe+: now also RP_LIM1.2
- net Probe-: now also RP_B1.2
- net RP_A+ renamed HVSW+
- net HVSW+: now also RP_LIM1.1
Other:
- removed sheet Resistor Networks
Changed lines of the file:
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@@
 	(wire
 		(pts
-			(xy 247.65 137.16) (xy 246.38 137.16)
-		)
-		(stroke
-			(width 0)
-			(type default)
-		)
-	)
-	(wire
-		(pts
 			(xy 203.2 151.13) (xy 209.55 151.13)
 		)
@@
 	(wire
 		(pts
+			(xy 240.03 137.16) (xy 247.65 137.16)
+		)
+		(stroke
+			(width 0)
+			(type default)
+		)
+	)
+	(wire
+		(pts
 			(xy 110.49 81.28) (xy 118.11 81.28)
 		)
@@
 	(wire
 		(pts
-			(xy 224.79 137.16) (xy 226.06 137.16)
+			(xy 224.79 137.16) (xy 232.41 137.16)
 		)
 		(stroke
@@
 	(wire
 		(pts
-			(xy 201.93 119.38) (xy 203.2 119.38)
+			(xy 201.93 119.38) (xy 209.55 119.38)
 		)
 		(stroke
@@
 	(wire
 		(pts
-			(xy 223.52 119.38) (xy 224.79 119.38)
-		)
-		(stroke
-			(width 0)
-			(type default)
-		)
-	)
-	(wire
-		(pts
 			(xy 153.67 53.34) (xy 153.67 52.07)
 		)
@@
 	(wire
 		(pts
+			(xy 217.17 119.38) (xy 224.79 119.38)
+		)
+		(stroke
+			(width 0)
+			(type default)
+		)
+	)
+	(wire
+		(pts
 			(xy 229.87 151.13) (xy 232.41 151.13)
 		)
@@
 		)
 	)
-	(global_label "RP_A-"
-		(shape input)
-		(at 223.52 119.38 180)
-		(fields_autoplaced yes)
-		(effects
-			(font
-				(size 1.27 1.27)
-			)
-			(justify right)
-		)
-		(property "Intersheetrefs" "${INTERSHEET_REFS}"
-			(at 214.3662 119.38 0)
-			(effects
-				(font
-					(size 1.27 1.27)
-				)
-				(justify right)
-				(hide yes)
-			)
-		)
-	)
 	(global_label "PulseCS-"
 		(shape output)
@@
 		)
 	)
-	(global_label "RP_A+"
-		(shape output)
-		(at 203.2 119.38 0)
-		(fields_autoplaced yes)
-		(effects
-			(font
-				(size 1.27 1.27)
-			)
-			(justify left)
-		)
-		(property "Intersheetrefs" "${INTERSHEET_REFS}"
-			(at 212.3538 119.38 0)
-			(effects
-				(font
-					(size 1.27 1.27)
-				)
-				(justify left)
-				(hide yes)
-			)
-		)
-	)
 	(global_label "Probe-"
 		(shape passive)
@@
 		)
 	)
-	(global_label "RP_B-"
-		(shape input)
-		(at 226.06 137.16 0)
-		(fields_autoplaced yes)
-		(effects
-			(font
-				(size 1.27 1.27)
-			)
-			(justify left)
-		)
-		(property "Intersheetrefs" "${INTERSHEET_REFS}"
-			(at 235.2138 137.16 0)
-			(effects
-				(font
-					(size 1.27 1.27)
-				)
-				(justify left)
-				(hide yes)
-			)
-		)
-	)
 	(global_label "IntTrigP"
 		(shape input)
@@
 		)
 	)
-	(global_label "RP_B+"
-		(shape output)
-		(at 246.38 137.16 180)
-		(fields_autoplaced yes)
-		(effects
-			(font
-				(size 1.27 1.27)
-			)
-			(justify right)
-		)
-		(property "Intersheetrefs" "${INTERSHEET_REFS}"
-			(at 237.2262 137.16 0)
-			(effects
-				(font
-					(size 1.27 1.27)
-				)
-				(justify right)
-				(hide yes)
-			)
-		)
-	)
 	(symbol
 		(lib_id "Device:R")
@@
 	(symbol
 		(lib_id "Device:R")
+		(at 236.22 137.16 90)
+		(mirror x)
+		(unit 1)
+		(exclude_from_sim no)
+		(in_bom yes)
+		(on_board yes)
+		(dnp no)
+		(property "Reference" "RP_B1"
+			(at 236.22 142.24 90)
+			(effects
+				(font
+					(size 1.27 1.27)
+				)
+			)
+		)
+		(property "Value" "WSHP2818R0200FEA"
+			(at 236.22 139.7 90)
+			(effects
+				(font
+					(size 1.27 1.27)
+				)
+			)
+		)
+		(property "Footprint" "project-footprints:WSHP2818R0200FEA"
+			(at 236.22 135.382 90)
+			(effects
+				(font
+					(size 1.27 1.27)
+				)
+				(hide yes)
+			)
+		)
+		(property "Datasheet" "https://jlcpcb.com/api/file/downloadByFileSystemAccessId/8589815038384517120"
+			(at 236.22 137.16 0)
+			(effects
+				(font
+					(size 1.27 1.27)
+				)
+				(hide yes)
+			)
+		)
+		(property "Description" "Resistor"
+			(at 236.22 137.16 0)
+			(effects
+				(font
+					(size 1.27 1.27)
+				)
+				(hide yes)
+			)
+		)
+		(pin "2"
+		)
+		(pin "1"
+		)
+		(instances
+			(project "BitCrusher"
+				(path "/e1be550d-9ce6-42b1-a89a-c00b9d7586dd/a0344160-5a1e-4ade-9868-d857907b9d6d"
+					(reference "RP_B1")
+					(unit 1)
+				)
+			)
+		)
+	)
+	(symbol
+		(lib_id "Device:R")
 		(at 118.11 69.85 0)
 		(unit 1)
@@
 			)
 		)
-		(property "Footprint" "Capacitor_SMD:C_0402_1005Metric"
+		(property "Footprint" "Capacitor_SMD:C_0603_1608Metric"
 			(at 154.6352 52.07 0)
 			(effects
@@
 	)
 	(symbol
+		(lib_id "Device:R")
+		(at 213.36 119.38 90)
+		(unit 1)
+		(exclude_from_sim no)
+		(in_bom yes)
+		(on_board yes)
+		(dnp no)
+		(fields_autoplaced yes)
+		(property "Reference" "RP_LIM1"
+			(at 213.36 113.03 90)
+			(effects
+				(font
+					(size 1.27 1.27)
+				)
+			)
+		)
+		(property "Value" "PF2472-0R1F1"
+			(at 213.36 115.57 90)
+			(effects
+				(font
+					(size 1.27 1.27)
+				)
+			)
+		)
+		(property "Footprint" "Package_TO_SOT_THT:TO-247-2_Horizontal_TabDown"
+			(at 213.36 121.158 90)
+			(effects
+				(font
+					(size 1.27 1.27)
+				)
+				(hide yes)
+			)
+		)
+		(property "Datasheet" "~"
+			(at 213.36 119.38 0)
+			(effects
+				(font
+					(size 1.27 1.27)
+				)
+				(hide yes)
+			)
+		)
+		(property "Description" "Resistor"
+			(at 213.36 119.38 0)
+			(effects
+				(font
+					(size 1.27 1.27)
+				)
+				(hide yes)
+			)
+		)
+		(pin "2"
+		)
+		(pin "1"
+		)
+		(instances
+			(project "BitCrusher"
+				(path "/e1be550d-9ce6-42b1-a89a-c00b9d7586dd/a0344160-5a1e-4ade-9868-d857907b9d6d"
+					(reference "RP_LIM1")
+					(unit 1)
+				)
+			)
+		)
+	)
+	(symbol
 		(lib_id "Transistor_FET:GS66508B")
 		(at 193.04 76.2 0)
@@
 				)
 			)
-		)
-	)
-	(sheet
-		(at 250.825 144.145)
-		(size 32.385 19.05)
-		(exclude_from_sim no)
-		(in_bom yes)
-		(on_board yes)
-		(dnp no)
-		(fields_autoplaced yes)
-		(stroke
-			(width 0.1524)
-			(type solid)
-		)
-		(fill
-			(color 0 0 0 0.0000)
-		)
-		(property "Sheetname" "Resistor Networks"
-			(at 250.825 143.4334 0)
-			(effects
-				(font
-					(size 1.27 1.27)
-				)
-				(justify left bottom)
-			)
-		)
-		(property "Sheetfile" "resistor-networks.kicad_sch"
-			(at 250.825 163.7796 0)
-			(effects
-				(font
-					(size 1.27 1.27)
-				)
-				(justify left top)
-			)
-		)
-		(instances
-			(project "BitCrusher"
-				(path "/e1be550d-9ce6-42b1-a89a-c00b9d7586dd/a0344160-5a1e-4ade-9868-d857907b9d6d"
-					(page "6")
-				)
-			)

Commit message: More little fixes
Parts:
- C30: JLCPCB# (none) -> C60077
Changed lines of the file:
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@@
+			)
+		)
+		(property "JLCPCB#" "C60077"
+			(at 153.67 48.26 0)
+			(effects
+				(font
+					(size 1.27 1.27)
+				)
+				(hide yes)
 			)
 		)

Commit message: _
Parts:
- RP_LIM1: footprint Package_TO_SOT_THT:TO-247-2_Horizontal_TabDown -> project-footprints:TO-247-2_Horizontal_TabDown
Changed lines of the file:
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@@
 			)
 		)
-		(property "Footprint" "Package_TO_SOT_THT:TO-247-2_Horizontal_TabDown"
+		(property "Footprint" "project-footprints:TO-247-2_Horizontal_TabDown"
 			(at 213.36 121.158 90)
 			(effects
