File: flyback-converter-test/flyback-test.kicad_sch (KiCad schematic)
At the start: 20 parts, among them Q1 NMOS, U1 PUCC28C53DR

Commit message: _
Parts:
- removed C1: ${SIM.PARAMS}, symbol Device:C
- removed CT1: 1n, symbol Device:C
- removed Q1: NMOS, symbol Simulation_SPICE:NMOS
- removed RT1: 17k, symbol Device:R
- removed U1: PUCC28C53DR, D0008A-IPC_A, symbol project_lib:PUCC28C53DR
- removed VFB1: VPWL, symbol Simulation_SPICE:VPWL
- added C5: 0.1u, Capacitor_SMD:C_0402_1005Metric, symbol Device:C
- added D2: D, symbol Device:D
- added D5: 1N5819, Diode_SMD:D_SOD-323, symbol Device:D_Schottky
- added L1: 1u, symbol Device:L
- added Q1: Q_NMOS_DGS, Package_TO_SOT_SMD:TO-252-2, symbol Transistor_FET:Q_NMOS_DGS
- added Q2: 2SA1213, Package_TO_SOT_SMD:SOT-89-3, symbol Device:Q_PNP
- added R3: 10, Resistor_SMD:R_0805_2012Metric, symbol Device:R
- added R4: 5, Resistor_SMD:R_0805_2012Metric, symbol Device:R
- added R5: 1, symbol Device:R
- added U2: UCC27511ADBV, Package_TO_SOT_SMD:SOT-23-6, symbol Driver_FET:UCC27511ADBV
- added V2: VPULSE, symbol Simulation_SPICE:VPULSE
Connections:
- net 0: now also R5.2
- net GND: now also C5.1, L1.1, Q2.C, U2.4 (GND), U2.5 (IN-), V2.2
- net Vin: now also C5.2, D2.2 (A), U2.1 (V_{DD}); no longer C2.1, C3.1, C4.1, R2.1
- net at R_CS1.1, R_CSF1.2: now also Q1.3 (S)
- net at LP1.2: now also Q1.1 (D)
- new net: C2.1, C3.1, C4.1, D2.1 (K), R2.1
- new net: D5.1 (K), Q1.2 (G), R4.2
- new net: L1.2, R5.1
- new net: U2.6 (IN+), V2.1
- new net: D5.2 (A), Q2.B, R3.2, U2.3 (OUTL)
- new net: R3.1, U2.2 (OUTH)
- new net: Q2.E, R4.1
Other:
- note removed: "CS must not exceed 1V during normal operation. Current limit hit at CS=1V"
- note removed: "Error Amp Input (from SS)"
- note removed: "Error Amp Output"
- note removed: "Internal Reference Output"
- note removed: "Oscillator RC"
- note removed: "Oscillator RtCt (100KHz)"
- note removed: "PS Current Sense"
- note removed: "PWM Gate Drive"
- note removed: "Vref Filter"
- moved on the sheet: C2, C3, C4

Commit message: more flyback sim work
Parts:
- removed C2, C3: 4.7u, symbol Device:C
- removed L1: 1u, symbol Device:L
- removed R5: 1, symbol Device:R
- added R7: 10, Resistor_SMD:R_0805_2012Metric, symbol Device:R
Connections:
- net 0 is gone; now on net GND: Cout1.2, LS1.1, Rload1.2
- net at D5.2 (A), Q2.B, R3.2: now also R7.2; no longer U2.3 (OUTL)
- net Vin renamed VDD
- new net: R7.1, U2.3 (OUTL)

Commit message: no sim errors now
Parts:
- added R6: 1, Resistor_SMD:R_0805_2012Metric, symbol Device:R
Connections:
- net at D5.1 (K), R4.2: now also R6.2; no longer Q1.2 (G)
- new net: Q1.2 (G), R6.1
Changed lines of the file:
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@@
 	(wire
 		(pts
-			(xy 177.8 85.09) (xy 177.8 87.63)
+			(xy 177.8 85.09) (xy 177.8 97.79)
 		)
 		(stroke
@@
 	(wire
 		(pts
-			(xy 177.8 64.77) (xy 205.74 64.77)
+			(xy 177.8 64.77) (xy 186.69 64.77)
 		)
 		(stroke
@@
 	(wire
 		(pts
+			(xy 194.31 64.77) (xy 205.74 64.77)
+		)
+		(stroke
+			(width 0)
+			(type default)
+		)
+	)
+	(wire
+		(pts
 			(xy 186.69 33.02) (xy 186.69 31.75)
 		)
@@
 	)
 	(symbol
+		(lib_id "Device:R")
+		(at 190.5 64.77 270)
+		(unit 1)
+		(exclude_from_sim no)
+		(in_bom yes)
+		(on_board yes)
+		(dnp no)
+		(fields_autoplaced yes)
+		(property "Reference" "R6"
+			(at 190.5 58.42 90)
+			(effects
+				(font
+					(size 1.27 1.27)
+				)
+			)
+		)
+		(property "Value" "1"
+			(at 190.5 60.96 90)
+			(effects
+				(font
+					(size 1.27 1.27)
+				)
+			)
+		)
+		(property "Footprint" "Resistor_SMD:R_0805_2012Metric"
+			(at 190.5 62.992 90)
+			(effects
+				(font
+					(size 1.27 1.27)
+				)
+				(hide yes)
+			)
+		)
+		(property "Datasheet" "~"
+			(at 190.5 64.77 0)
+			(effects
+				(font
+					(size 1.27 1.27)
+				)
+				(hide yes)
+			)
+		)
+		(property "Description" "Resistor"
+			(at 190.5 64.77 0)
+			(effects
+				(font
+					(size 1.27 1.27)
+				)
+				(hide yes)
+			)
+		)
+		(property "KLC_S4.2_3V3OUT" ""
+			(at 190.5 64.77 90)
+			(effects
+				(font
+					(size 1.27 1.27)
+				)
+				(hide yes)
+			)
+		)
+		(property "KLC_S4.2_VCC" ""
+			(at 190.5 64.77 90)
+			(effects
+				(font
+					(size 1.27 1.27)
+				)
+				(hide yes)
+			)
+		)
+		(pin "1"
+		)
+		(pin "2"
+		)
+		(instances
+			(project "flyback-test"
+				(path "/0e3fdada-5b30-4d9e-bef7-775c86a4f788"
+					(reference "R6")
+					(unit 1)
+				)
+			)
+		)
+	)
+	(symbol
 		(lib_id "Device:D")
 		(at 172.72 31.75 180)
@@
 	(symbol
 		(lib_id "power:GND")
-		(at 177.8 87.63 0)
+		(at 177.8 97.79 0)
 		(unit 1)
 		(exclude_from_sim no)
@@
 		(fields_autoplaced yes)
 		(property "Reference" "#PWR016"
-			(at 177.8 93.98 0)
+			(at 177.8 104.14 0)
 			(effects
 				(font
@@
 		)
 		(property "Value" "GND"
-			(at 177.8 92.71 0)
+			(at 177.8 102.87 0)
 			(effects
 				(font
@@
 		)
 		(property "Footprint" ""
-			(at 177.8 87.63 0)
+			(at 177.8 97.79 0)
 			(effects
 				(font
@@
 		)
 		(property "Datasheet" ""
-			(at 177.8 87.63 0)
+			(at 177.8 97.79 0)
 			(effects
 				(font
@@
 		)
 		(property "Description" "Power symbol creates a global label with name \"GND\" , ground"
-			(at 177.8 87.63 0)
+			(at 177.8 97.79 0)
 			(effects
 				(font
@@
 			(at 226.06 31.75 0)
 			(effects
+				(font
+					(size 1.27 1.27)
+				)
+				(hide yes)
+			)
+		)
+		(property "Sim.Params" "rs=0.01"
+			(at 226.06 31.75 0)
+			(effects
